File: IDA_demoprojekt/IDA_demoprojekt.kicad_pcb (KiCad board)
At the start: 4 copper layers, 61 x 29 mm, 28 parts, among them J1 USB_B_Micro, J2 Conn_Coaxial, J3 Conn_02x05_Odd_Even, U1 USBLC6-2SC6, U2 nRF24L01P, U3 AP2112K-3.3, U4 STM32L072KZTx, Y1 ASA-16.000MHZ-L-T

Commit message: tilføjet eksempler
Routing:
- added copper zone on B.Cu, net GND
- added copper zone on F.Cu, net GND
Other:
- board text added: "(c) Gert Lauritsen"
